Commit message: Enhanced train pipeline

File: urdf/core_bipedal_robot.urdf.xacro (robot description, xacro)
@@ -68,15 +68,17 @@
             </inertial>
         </link>
-        <joint name="${name}_hip_joint" type="continuous">
+        <joint name="${name}_hip_joint" type="revolute">
             <parent link="base_link"/>
             <child link="${name}_thigh"/>
             <origin xyz="0 ${shift} -0.5" rpy="0 0 0"/>
             <axis xyz="0 1 0"/>
+            <limit lower="-1.57" upper="1.57" effort="50" velocity="0.5"/>
         </joint>
-        <joint name="${name}_knee_joint" type="continuous">
+        <joint name="${name}_knee_joint" type="revolute">
             <parent link="${name}_thigh"/>
             <child link="${name}_shin"/>
             <origin xyz="0 0 -1" rpy="0 0 0"/>
             <axis xyz="0 1 0"/>
+            <limit lower="0.0" upper="1.57" effort="50" velocity="0.5"/>
         </joint>
 	</xacro:macro>

File: urdf/gazebo_bipedal_robot.urdf.xacro (robot description, xacro)
@@ -32,5 +32,5 @@
 	    <plugin name="joint_state_publisher" filename="libgazebo_ros_joint_state_publisher.so">
             <jointName>left_knee_joint, left_knee_joint, right_hip_joint, right_knee_joint</jointName>
-            <updateRate>50.0</updateRate>
+            <updateRate>60.0</updateRate>
             <alwaysOn>true</alwaysOn>
 	    </plugin>

Commit message: Evironment fix

File: urdf/core_bipedal_robot.urdf.xacro (robot description, xacro)
@@ -20,5 +20,5 @@
             <mass value="1.0"/>
 		    <origin xyz="0 0 0"/>
-		    <inertia ixx="0.1" ixy="0.0" ixz="0.0" iyy="0.1" iyz="0.0" izz="0.1"/>
+		    <inertia ixx="0.1" ixy="0.0001" ixz="0.0001" iyy="0.1" iyz="0.0001" izz="0.1"/>
 		</inertial>
 	</link>
@@ -43,5 +43,5 @@
                 <mass value="1.0"/>
                 <origin xyz="0 0 0"/>
-                <inertia ixx="0.1" ixy="0.0" ixz="0.0" iyy="0.1" iyz="0.0" izz="0.1"/>
+                <inertia ixx="0.1" ixy="0.0001" ixz="0.0001" iyy="0.1" iyz="0.0001" izz="0.1"/>
             </inertial>
         </link>
@@ -65,5 +65,5 @@
                 <mass value="1.0"/>
                 <origin xyz="0 0 0"/>
-                <inertia ixx="0.1" ixy="0.0" ixz="0.0" iyy="0.1" iyz="0.0" izz="0.1"/>
+                <inertia ixx="0.1" ixy="0.0001" ixz="0.0001" iyy="0.1" iyz="0.0001" izz="0.1"/>
             </inertial>
         </link>
@@ -73,5 +73,5 @@
             <origin xyz="0 ${shift} -0.5" rpy="0 0 0"/>
             <axis xyz="0 1 0"/>
-            <limit lower="-1.57" upper="1.57" effort="50" velocity="0.5"/>
+            <limit lower="-1.57" upper="1.57" effort="10" velocity="1"/>
         </joint>
         <joint name="${name}_knee_joint" type="revolute">
@@ -80,5 +80,5 @@
             <origin xyz="0 0 -1" rpy="0 0 0"/>
             <axis xyz="0 1 0"/>
-            <limit lower="0.0" upper="1.57" effort="50" velocity="0.5"/>
+            <limit lower="0.0" upper="1.57" effort="10" velocity="1"/>
         </joint>
 	</xacro:macro>

Commit message: Started adding parallel training

File: urdf/core_bipedal_robot.urdf.xacro (robot description, xacro)
@@ -5,5 +5,5 @@
 			<origin xyz="0 0 0" rpy="0 0 0"/>
 			<geometry>
-				<box size="1 1 1" />
+				<box size="0.75 1 1" />
 			</geometry>
 			<material name="blue">
@@ -11,15 +11,20 @@
 			</material>
 		</visual>
-		<collision>
+		<collision name="base_link">
 		    <origin xyz="0 0 0" rpy="0 0 0"/>
 			<geometry>
-				<box size="1 1 1" />
+				<box size="0.75 1 1" />
 			</geometry>
 		</collision>
 		<inertial>
-            <mass value="1.0"/>
+            <mass value="0.5"/>
 		    <origin xyz="0 0 0"/>
-		    <inertia ixx="0.1" ixy="0.0001" ixz="0.0001" iyy="0.1" iyz="0.0001" izz="0.1"/>
+		    <inertia ixx="0.1" ixy="0.0" ixz="0.0" iyy="0.1" iyz="0.0" izz="0.1"/>
 		</inertial>
+		<sensor name='base_link_contact' type='contact'>
+            <contact>
+                <collision>base_link</collision>
+            </contact>
+        </sensor>
 	</link>
 	<xacro:macro name="leg" params="name shift">
@@ -34,5 +39,5 @@
                 </material>
             </visual>
-            <collision>
+            <collision name="${name}_thigh_collision">
                 <origin xyz="0 0 -0.5" rpy="0 0 0"/>
                 <geometry>
@@ -41,7 +46,7 @@
             </collision>
             <inertial>
-                <mass value="1.0"/>
+                <mass value="1.5"/>
                 <origin xyz="0 0 0"/>
-                <inertia ixx="0.1" ixy="0.0001" ixz="0.0001" iyy="0.1" iyz="0.0001" izz="0.1"/>
+                <inertia ixx="0.1" ixy="0.0" ixz="0.0" iyy="0.1" iyz="0.0" izz="0.1"/>
             </inertial>
         </link>
@@ -56,5 +61,5 @@
                 </material>
             </visual>
-            <collision>
+            <collision name="${name}_shin_collision">
                 <origin xyz="0 0 -0.5" rpy="0 0 0"/>
                 <geometry>
@@ -63,7 +68,7 @@
             </collision>
             <inertial>
-                <mass value="1.0"/>
+                <mass value="0.6"/>
                 <origin xyz="0 0 0"/>
-                <inertia ixx="0.1" ixy="0.0001" ixz="0.0001" iyy="0.1" iyz="0.0001" izz="0.1"/>
+                <inertia ixx="0.1" ixy="0.0" ixz="0.0" iyy="0.1" iyz="0.0" izz="0.1"/>
             </inertial>
         </link>
@@ -73,5 +78,6 @@
             <origin xyz="0 ${shift} -0.5" rpy="0 0 0"/>
             <axis xyz="0 1 0"/>
-            <limit lower="-1.57" upper="1.57" effort="10" velocity="1"/>
+            <limit lower="-1.57" upper="1.57" effort="50" velocity="1"/>
+            <dynamics damping="0.01" friction="0.02"/>
         </joint>
         <joint name="${name}_knee_joint" type="revolute">
@@ -80,5 +86,6 @@
             <origin xyz="0 0 -1" rpy="0 0 0"/>
             <axis xyz="0 1 0"/>
-            <limit lower="0.0" upper="1.57" effort="10" velocity="1"/>
+            <limit lower="0.0" upper="1.57" effort="30" velocity="1"/>
+            <dynamics damping="0.01" friction="0.02"/>
         </joint>
 	</xacro:macro>

File: urdf/gazebo_bipedal_robot.urdf.xacro (robot description, xacro)
@@ -23,16 +23,3 @@
 	<xacro:transmission joint="right_hip_joint"/>
 	<xacro:transmission joint="right_knee_joint"/>
-	<gazebo>
-	    <plugin name="gazebo_ros_control" filename="libgazebo_ros_control.so">
-	        <controlPeriod>0.001</controlPeriod>
-	        <legacyModeNS>true</legacyModeNS>
-	        <robotNamespace>/bipedal_robot</robotNamespace>
-	        <robotSimType>gazebo_ros_control/DefaultRobotHWSim</robotSimType>
-	    </plugin>
-	    <plugin name="joint_state_publisher" filename="libgazebo_ros_joint_state_publisher.so">
-            <jointName>left_knee_joint, left_knee_joint, right_hip_joint, right_knee_joint</jointName>
-            <updateRate>60.0</updateRate>
-            <alwaysOn>true</alwaysOn>
-	    </plugin>
-	</gazebo>
 </robot>

Commit message: Changed urdf file

File: urdf/core_bipedal_robot.urdf.xacro (robot description, xacro)
@@ -5,5 +5,5 @@
 			<origin xyz="0 0 0" rpy="0 0 0"/>
 			<geometry>
-				<box size="0.75 1 1" />
+				<box size="0.05 0.08 0.08" />
 			</geometry>
 			<material name="blue">
@@ -14,24 +14,19 @@
 		    <origin xyz="0 0 0" rpy="0 0 0"/>
 			<geometry>
-				<box size="0.75 1 1" />
+				<box size="0.05 0.08 0.08" />
 			</geometry>
 		</collision>
 		<inertial>
-            <mass value="0.5"/>
+            <mass value="0.16"/>
 		    <origin xyz="0 0 0"/>
 		    <inertia ixx="0.1" ixy="0.0" ixz="0.0" iyy="0.1" iyz="0.0" izz="0.1"/>
 		</inertial>
-		<sensor name='base_link_contact' type='contact'>
-            <contact>
-                <collision>base_link</collision>
-            </contact>
-        </sensor>
 	</link>
 	<xacro:macro name="leg" params="name shift">
         <link name="${name}_thigh">
             <visual>
-                <origin xyz="0 0 -0.5" rpy="0 0 0"/>
+                <origin xyz="0 0 -0.05" rpy="0 0 0"/>
                 <geometry>
-                    <box size="0.25 0.25 1" />
+                    <cylinder radius="0.01" length="0.1"/>
                 </geometry>
                 <material name="blue">
@@ -40,11 +35,11 @@
             </visual>
             <collision name="${name}_thigh_collision">
-                <origin xyz="0 0 -0.5" rpy="0 0 0"/>
+                <origin xyz="0 0 -0.05" rpy="0 0 0"/>
                 <geometry>
-                    <box size="0.25 0.25 1" />
+                    <cylinder radius="0.01" length="0.1"/>
                 </geometry>
             </collision>
             <inertial>
-                <mass value="1.5"/>
+                <mass value="0.16"/>
                 <origin xyz="0 0 0"/>
                 <inertia ixx="0.1" ixy="0.0" ixz="0.0" iyy="0.1" iyz="0.0" izz="0.1"/>
@@ -53,7 +48,7 @@
         <link name="${name}_shin">
             <visual>
-                <origin xyz="0 0 -0.5" rpy="0 0 0"/>
+                <origin xyz="0 0 -0.05" rpy="0 0 0"/>
                 <geometry>
-                    <box size="0.25 0.25 1" />
+                    <cylinder radius="0.01" length="0.1"/>
                 </geometry>
                 <material name="blue">
@@ -62,11 +57,33 @@
             </visual>
             <collision name="${name}_shin_collision">
-                <origin xyz="0 0 -0.5" rpy="0 0 0"/>
+                <origin xyz="0 0 -0.05" rpy="0 0 0"/>
                 <geometry>
-                    <box size="0.25 0.25 1" />
+                    <cylinder radius="0.01" length="0.1"/>
                 </geometry>
             </collision>
             <inertial>
-                <mass value="0.6"/>
+                <mass value="0.16"/>
+                <origin xyz="0 0 0"/>
+                <inertia ixx="0.1" ixy="0.0" ixz="0.0" iyy="0.1" iyz="0.0" izz="0.1"/>
+            </inertial>
+        </link>
+        <link name="${name}_foot">
+            <visual>
+                <origin xyz="0 0 -0.005" rpy="0 0 0"/>
+                <geometry>
+                    <box size="0.05 0.04 0.01" />
+                </geometry>
+                <material name="blue">
+                    <color rgba="0 0 1 1"/>
+                </material>
+            </visual>
+            <collision name="${name}_foot_collision">
+                <origin xyz="0 0 -0.005" rpy="0 0 0"/>
+                <geometry>
+                    <box size="0.05 0.04 0.01" />
+                </geometry>
+            </collision>
+            <inertial>
+                <mass value="0.02"/>
                 <origin xyz="0 0 0"/>
                 <inertia ixx="0.1" ixy="0.0" ixz="0.0" iyy="0.1" iyz="0.0" izz="0.1"/>
@@ -76,19 +93,27 @@
             <parent link="base_link"/>
             <child link="${name}_thigh"/>
-            <origin xyz="0 ${shift} -0.5" rpy="0 0 0"/>
+            <origin xyz="0 ${shift} -0.04" rpy="0 0 0"/>
             <axis xyz="0 1 0"/>
-            <limit lower="-1.57" upper="1.57" effort="50" velocity="1"/>
-            <dynamics damping="0.01" friction="0.02"/>
+            <limit lower="-1.57" upper="1.57" effort="30" velocity="1.5"/>
+            <dynamics damping="0.5" friction="0.3"/>
         </joint>
         <joint name="${name}_knee_joint" type="revolute">
             <parent link="${name}_thigh"/>
             <child link="${name}_shin"/>
-            <origin xyz="0 0 -1" rpy="0 0 0"/>
+            <origin xyz="0 0 -0.1" rpy="0 0 0"/>
             <axis xyz="0 1 0"/>
             <limit lower="0.0" upper="1.57" effort="30" velocity="1"/>
-            <dynamics damping="0.01" friction="0.02"/>
+            <dynamics damping="0.5" friction="0.3"/>
+        </joint>
+        <joint name="${name}_ankle_joint" type="revolute">
+            <parent link="${name}_shin"/>
+            <child link="${name}_foot"/>
+            <origin xyz="0 0 -0.1" rpy="0 0 0"/>
+            <axis xyz="0 1 0"/>
+            <limit lower="-1.57" upper="1.57" effort="30" velocity="1"/>
+            <dynamics damping="0.5" friction="0.3"/>
         </joint>
 	</xacro:macro>
-	<xacro:leg name="left" shift="0.5"/>
-	<xacro:leg name="right" shift="-0.5"/>
+	<xacro:leg name="left" shift="0.04"/>
+	<xacro:leg name="right" shift="-0.04"/>
 </robot>

File: urdf/gazebo_bipedal_robot.urdf.xacro (robot description, xacro)
@@ -8,5 +8,5 @@
     </joint>
 	<xacro:macro name="transmission" params="joint">
-        <transmission name="transmission1">
+        <transmission name="${joint}_transmission">
             <type>transmission_interface/SimpleTransmission</type>
             <joint name="${joint}">

Commit message: Added new joints, added contact plugin

File: urdf/core_bipedal_robot.urdf.xacro (robot description, xacro)
@@ -24,4 +24,11 @@
 	</link>
 	<xacro:macro name="leg" params="name shift">
+	    <link name="${name}_hip_link">
+	        <inertial>
+                <mass value="0.01"/>
+                <origin xyz="0 0 0"/>
+                <inertia ixx="0.1" ixy="0.0" ixz="0.0" iyy="0.1" iyz="0.0" izz="0.1"/>
+            </inertial>
+	    </link>
         <link name="${name}_thigh">
             <visual>
@@ -68,4 +75,11 @@
             </inertial>
         </link>
+        <link name="${name}_ankle_link">
+            <inertial>
+                <mass value="0.01"/>
+                <origin xyz="0 0 0"/>
+                <inertia ixx="0.1" ixy="0.0" ixz="0.0" iyy="0.1" iyz="0.0" izz="0.1"/>
+            </inertial>
+        </link>
         <link name="${name}_foot">
             <visual>
@@ -90,10 +104,18 @@
             </inertial>
         </link>
-        <joint name="${name}_hip_joint" type="revolute">
+        <joint name="${name}_hip_joint1" type="revolute">
             <parent link="base_link"/>
+            <child link="${name}_hip_link"/>
+            <origin xyz="0 ${shift} -0.03" rpy="0 0 0"/>
+            <axis xyz="1 0 0"/>
+            <limit lower="-1.57" upper="1.57" effort="20" velocity="1.5"/>
+            <dynamics damping="0.5" friction="0.3"/>
+        </joint>
+        <joint name="${name}_hip_joint2" type="revolute">
+            <parent link="${name}_hip_link"/>
             <child link="${name}_thigh"/>
-            <origin xyz="0 ${shift} -0.04" rpy="0 0 0"/>
+            <origin xyz="0 0 -0.03" rpy="0 0 0"/>
             <axis xyz="0 1 0"/>
-            <limit lower="-1.57" upper="1.57" effort="30" velocity="1.5"/>
+            <limit lower="-1.57" upper="1.57" effort="20" velocity="1.5"/>
             <dynamics damping="0.5" friction="0.3"/>
         </joint>
@@ -103,13 +125,21 @@
             <origin xyz="0 0 -0.1" rpy="0 0 0"/>
             <axis xyz="0 1 0"/>
-            <limit lower="0.0" upper="1.57" effort="30" velocity="1"/>
+            <limit lower="0.0" upper="1.57" effort="20" velocity="1"/>
             <dynamics damping="0.5" friction="0.3"/>
         </joint>
-        <joint name="${name}_ankle_joint" type="revolute">
+        <joint name="${name}_ankle_joint1" type="revolute">
             <parent link="${name}_shin"/>
+            <child link="${name}_ankle_link"/>
+            <origin xyz="0 0 -0.1" rpy="0 0 0"/>
+            <axis xyz="0 1 0"/>
+            <limit lower="-1.57" upper="1.57" effort="20" velocity="1"/>
+            <dynamics damping="0.5" friction="0.3"/>
+        </joint>
+        <joint name="${name}_ankle_joint2" type="revolute">
+            <parent link="${name}_ankle_link"/>
             <child link="${name}_foot"/>
             <origin xyz="0 0 -0.1" rpy="0 0 0"/>
-            <axis xyz="0 1 0"/>
-            <limit lower="-1.57" upper="1.57" effort="30" velocity="1"/>
+            <axis xyz="1 0 0"/>
+            <limit lower="-1.57" upper="1.57" effort="20" velocity="1"/>
             <dynamics damping="0.5" friction="0.3"/>
         </joint>

File: urdf/full_bipedal_robot.urdf (robot description, URDF)
Before this commit: robot bipedal_robot, 6 links, 5 joints
Links:
- added link left_ankle_link, mass 0.01
- added link left_foot, mass 0.02; collision box size=0.05 0.04 0.01; visual box size=0.05 0.04 0.01
- added link left_hip_link, mass 0.01
- added link right_ankle_link, mass 0.01
- added link right_foot, mass 0.02; collision box size=0.05 0.04 0.01; visual box size=0.05 0.04 0.01
- added link right_hip_link, mass 0.01
- link base_link: mass 0.5 -> 0.16; geometry collision box size=0.05 0.08 0.08; visual box size=0.05 0.08 0.08
- link left_shin: mass 0.6 -> 0.16; geometry collision cylinder length=0.1 radius=0.01; visual cylinder length=0.1 radius=0.01
- link left_thigh: mass 1.5 -> 0.16; geometry collision cylinder length=0.1 radius=0.01; visual cylinder length=0.1 radius=0.01
- link right_shin: mass 0.6 -> 0.16; geometry collision cylinder length=0.1 radius=0.01; visual cylinder length=0.1 radius=0.01
- link right_thigh: mass 1.5 -> 0.16; geometry collision cylinder length=0.1 radius=0.01; visual cylinder length=0.1 radius=0.01
Joints:
- removed joint left_hip_joint
- removed joint right_hip_joint
- added joint left_ankle_joint1: type revolute, parent left_shin, child left_ankle_link, origin xyz=0 0 -0.1 rpy=0 0 0, axis 0 1 0, limit lower=-1.57 upper=1.57 effort=20 velocity=1
- added joint left_ankle_joint2: type revolute, parent left_ankle_link, child left_foot, origin xyz=0 0 -0.1 rpy=0 0 0, axis 1 0 0, limit lower=-1.57 upper=1.57 effort=20 velocity=1
- added joint left_hip_joint1: type revolute, parent base_link, child left_hip_link, origin xyz=0 0.04 -0.03 rpy=0 0 0, axis 1 0 0, limit lower=-1.57 upper=1.57 effort=20 velocity=1.5
- added joint left_hip_joint2: type revolute, parent left_hip_link, child left_thigh, origin xyz=0 0 -0.03 rpy=0 0 0, axis 0 1 0, limit lower=-1.57 upper=1.57 effort=20 velocity=1.5
- added joint right_ankle_joint1: type revolute, parent right_shin, child right_ankle_link, origin xyz=0 0 -0.1 rpy=0 0 0, axis 0 1 0, limit lower=-1.57 upper=1.57 effort=20 velocity=1
- added joint right_ankle_joint2: type revolute, parent right_ankle_link, child right_foot, origin xyz=0 0 -0.1 rpy=0 0 0, axis 1 0 0, limit lower=-1.57 upper=1.57 effort=20 velocity=1
- added joint right_hip_joint1: type revolute, parent base_link, child right_hip_link, origin xyz=0 -0.04 -0.03 rpy=0 0 0, axis 1 0 0, limit lower=-1.57 upper=1.57 effort=20 velocity=1.5
- added joint right_hip_joint2: type revolute, parent right_hip_link, child right_thigh, origin xyz=0 0 -0.03 rpy=0 0 0, axis 0 1 0, limit lower=-1.57 upper=1.57 effort=20 velocity=1.5
- joint left_knee_joint: limit lower=0.0 upper=1.57 effort=30 velocity=1 -> lower=0.0 upper=1.57 effort=20 velocity=1; origin xyz=0 0 -1 rpy=0 0 0 -> xyz=0 0 -0.1 rpy=0 0 0
- joint right_knee_joint: limit lower=0.0 upper=1.57 effort=30 velocity=1 -> lower=0.0 upper=1.57 effort=20 velocity=1; origin xyz=0 0 -1 rpy=0 0 0 -> xyz=0 0 -0.1 rpy=0 0 0

File: urdf/gazebo_bipedal_robot.urdf.xacro (robot description, xacro)
@@ -19,15 +19,14 @@
         </transmission>
 	</xacro:macro>
-	<xacro:transmission joint="left_hip_joint"/>
+	<xacro:transmission joint="left_hip_joint1"/>
+	<xacro:transmission joint="left_hip_joint2"/>
 	<xacro:transmission joint="left_knee_joint"/>
-	<xacro:transmission joint="right_hip_joint"/>
+	<xacro:transmission joint="left_ankle_joint1"/>
+	<xacro:transmission joint="left_ankle_joint2"/>
+	<xacro:transmission joint="right_hip_joint1"/>
+	<xacro:transmission joint="right_hip_joint2"/>
 	<xacro:transmission joint="right_knee_joint"/>
-	<!-- <gazebo>
-        <plugin name="joint_state_publisher" filename="libgazebo_ros_joint_state_publisher.so">
-            <jointName>left_hip_joint, left_knee_joint, right_hip_joint, right_knee_joint</jointName>
-            <updateRate>50.0</updateRate>
-            <alwaysOn>true</alwaysOn>
-        </plugin>
-    </gazebo> -->
+	<xacro:transmission joint="right_ankle_joint1"/>
+	<xacro:transmission joint="right_ankle_joint2"/>
     <gazebo>
         <plugin name="gazebo_ros_control" filename="libgazebo_ros_control.so">
@@ -35,3 +34,15 @@
         </plugin>
     </gazebo>
+    <gazebo reference="left_foot">
+        <sensor name="left_foot_sensor" type="contact">
+            <always_on>true</always_on>
+            <contact>
+                <collision>left_foot_collision_collision</collision>
+            </contact>
+            <plugin name="left_foot_plugin" filename="libgazebo_ros_bumper.so">
+                <bumperTopicName>left_foot_contact</bumperTopicName>
+                <frameName>left_foot</frameName>
+            </plugin>
+        </sensor>
+    </gazebo>
 </robot>
