Commit message: Modified limits of new joints

File: urdf/core_bipedal_robot.urdf.xacro (robot description, xacro)
@@ -23,5 +23,5 @@
 		</inertial>
 	</link>
-	<xacro:macro name="leg" params="name shift">
+	<xacro:macro name="leg" params="name shift hip_left_limit hip_right_limit">
 	    <link name="${name}_hip_link">
 	        <inertial>
@@ -49,5 +49,5 @@
             <inertial>
                 <mass value="0.16"/>
-                <origin xyz="0 0 0"/>
+                <origin xyz="0 0 -0.05"/>
                 <inertia ixx="0.1" ixy="0.0" ixz="0.0" iyy="0.1" iyz="0.0" izz="0.1"/>
             </inertial>
@@ -71,5 +71,5 @@
             <inertial>
                 <mass value="0.16"/>
-                <origin xyz="0 0 0"/>
+                <origin xyz="0 0 -0.05"/>
                 <inertia ixx="0.1" ixy="0.0" ixz="0.0" iyy="0.1" iyz="0.0" izz="0.1"/>
             </inertial>
@@ -100,5 +100,5 @@
             <inertial>
                 <mass value="0.02"/>
-                <origin xyz="0 0 0"/>
+                <origin xyz="0 0 -0.005"/>
                 <inertia ixx="0.1" ixy="0.0" ixz="0.0" iyy="0.1" iyz="0.0" izz="0.1"/>
             </inertial>
@@ -109,5 +109,5 @@
             <origin xyz="0 ${shift} -0.03" rpy="0 0 0"/>
             <axis xyz="1 0 0"/>
-            <limit lower="-1.57" upper="1.57" effort="20" velocity="1.5"/>
+            <limit lower="${hip_left_limit}" upper="${hip_right_limit}" effort="20" velocity="1.5"/>
             <dynamics damping="0.5" friction="0.3"/>
         </joint>
@@ -115,5 +115,5 @@
             <parent link="${name}_hip_link"/>
             <child link="${name}_thigh"/>
-            <origin xyz="0 0 -0.03" rpy="0 0 0"/>
+            <origin xyz="0 0 0" rpy="0 0 0"/>
             <axis xyz="0 1 0"/>
             <limit lower="-1.57" upper="1.57" effort="20" velocity="1.5"/>
@@ -133,5 +133,5 @@
             <origin xyz="0 0 -0.1" rpy="0 0 0"/>
             <axis xyz="0 1 0"/>
-            <limit lower="-1.57" upper="1.57" effort="20" velocity="1"/>
+            <limit lower="-1.05" upper="0.52" effort="20" velocity="1"/>
             <dynamics damping="0.5" friction="0.3"/>
         </joint>
@@ -139,11 +139,11 @@
             <parent link="${name}_ankle_link"/>
             <child link="${name}_foot"/>
-            <origin xyz="0 0 -0.1" rpy="0 0 0"/>
+            <origin xyz="0 0 0" rpy="0 0 0"/>
             <axis xyz="1 0 0"/>
-            <limit lower="-1.57" upper="1.57" effort="20" velocity="1"/>
+            <limit lower="-0.52" upper="0.52" effort="20" velocity="1"/>
             <dynamics damping="0.5" friction="0.3"/>
         </joint>
 	</xacro:macro>
-	<xacro:leg name="left" shift="0.04"/>
-	<xacro:leg name="right" shift="-0.04"/>
+	<xacro:leg name="left" shift="0.04" hip_left_limit="-0.26" hip_right_limit="0.78"/>
+	<xacro:leg name="right" shift="-0.04" hip_left_limit="-0.78" hip_right_limit="0.26"/>
 </robot>

Commit message: Modified main urdf file

File: urdf/core_bipedal_robot.urdf.xacro (robot description, xacro)
@@ -1,9 +1,15 @@
 <?xml version="1.0"?>
 <robot name="bipedal_robot" xmlns:xacro="http://www.ros.org/wiki/xacro">
+    <xacro:property name="torso_height" value="0.7"/>
+    <xacro:property name="torso_width" value="0.7"/>
+    <xacro:property name="thigh_len" value="0.6"/>
+    <xacro:property name="shin_len" value="0.6"/>
+    <xacro:property name="foot_thickness" value="0.08"/>
+    <!-- Base link -->
 	<link name="base_link">
 		<visual>
 			<origin xyz="0 0 0" rpy="0 0 0"/>
 			<geometry>
-				<box size="0.05 0.08 0.08" />
+				<box size="0.3 ${torso_width} ${torso_height}"/>
 			</geometry>
 			<material name="blue">
@@ -14,13 +20,14 @@
 		    <origin xyz="0 0 0" rpy="0 0 0"/>
 			<geometry>
-				<box size="0.05 0.08 0.08" />
+				<box size="0.3 0.7 ${torso_height}"/>
 			</geometry>
 		</collision>
 		<inertial>
-            <mass value="0.16"/>
+            <mass value="1.5"/>
 		    <origin xyz="0 0 0"/>
 		    <inertia ixx="0.1" ixy="0.0" ixz="0.0" iyy="0.1" iyz="0.0" izz="0.1"/>
 		</inertial>
 	</link>
+	<!-- Leg links and joints -->
 	<xacro:macro name="leg" params="name shift hip_left_limit hip_right_limit">
 	    <link name="${name}_hip_link">
@@ -33,7 +40,7 @@
         <link name="${name}_thigh">
             <visual>
-                <origin xyz="0 0 -0.05" rpy="0 0 0"/>
+                <origin xyz="0 0 ${-thigh_len/2}" rpy="0 0 0"/>
                 <geometry>
-                    <cylinder radius="0.01" length="0.1"/>
+                    <cylinder radius="0.07" length="${thigh_len}"/>
                 </geometry>
                 <material name="blue">
@@ -42,12 +49,12 @@
             </visual>
             <collision name="${name}_thigh_collision">
-                <origin xyz="0 0 -0.05" rpy="0 0 0"/>
+                <origin xyz="0 0 ${-thigh_len/2}" rpy="0 0 0"/>
                 <geometry>
-                    <cylinder radius="0.01" length="0.1"/>
+                    <cylinder radius="0.07" length="${thigh_len}"/>
                 </geometry>
             </collision>
             <inertial>
-                <mass value="0.16"/>
-                <origin xyz="0 0 -0.05"/>
+                <mass value="2.5"/>
+                <origin xyz="0 0 0"/>
                 <inertia ixx="0.1" ixy="0.0" ixz="0.0" iyy="0.1" iyz="0.0" izz="0.1"/>
             </inertial>
@@ -55,7 +62,7 @@
         <link name="${name}_shin">
             <visual>
-                <origin xyz="0 0 -0.05" rpy="0 0 0"/>
+                <origin xyz="0 0 ${-shin_len/2}" rpy="0 0 0"/>
                 <geometry>
-                    <cylinder radius="0.01" length="0.1"/>
+                    <cylinder radius="0.07" length="${shin_len}"/>
                 </geometry>
                 <material name="blue">
@@ -64,12 +71,12 @@
             </visual>
             <collision name="${name}_shin_collision">
-                <origin xyz="0 0 -0.05" rpy="0 0 0"/>
+                <origin xyz="0 0 ${-shin_len/2}" rpy="0 0 0"/>
                 <geometry>
-                    <cylinder radius="0.01" length="0.1"/>
+                    <cylinder radius="0.07" length="${shin_len}"/>
                 </geometry>
             </collision>
             <inertial>
-                <mass value="0.16"/>
-                <origin xyz="0 0 -0.05"/>
+                <mass value="2"/>
+                <origin xyz="0 0 0"/>
                 <inertia ixx="0.1" ixy="0.0" ixz="0.0" iyy="0.1" iyz="0.0" izz="0.1"/>
             </inertial>
@@ -84,7 +91,7 @@
         <link name="${name}_foot">
             <visual>
-                <origin xyz="0 0 -0.005" rpy="0 0 0"/>
+                <origin xyz="0 0 ${-foot_thickness/2}" rpy="0 0 0"/>
                 <geometry>
-                    <box size="0.05 0.04 0.01" />
+                    <box size="0.45 0.3 ${foot_thickness}" />
                 </geometry>
                 <material name="blue">
@@ -93,12 +100,12 @@
             </visual>
             <collision name="${name}_foot_collision">
-                <origin xyz="0 0 -0.005" rpy="0 0 0"/>
+                <origin xyz="0 0 ${-foot_thickness/2}" rpy="0 0 0"/>
                 <geometry>
-                    <box size="0.05 0.04 0.01" />
+                    <box size="0.45 0.3 ${foot_thickness}" />
                 </geometry>
             </collision>
             <inertial>
-                <mass value="0.02"/>
-                <origin xyz="0 0 -0.005"/>
+                <mass value="1"/>
+                <origin xyz="0 0 0"/>
                 <inertia ixx="0.1" ixy="0.0" ixz="0.0" iyy="0.1" iyz="0.0" izz="0.1"/>
             </inertial>
@@ -107,8 +114,7 @@
             <parent link="base_link"/>
             <child link="${name}_hip_link"/>
-            <origin xyz="0 ${shift} -0.03" rpy="0 0 0"/>
+            <origin xyz="0 ${shift} ${-torso_height/2}" rpy="0 0 0"/>
             <axis xyz="1 0 0"/>
-            <limit lower="${hip_left_limit}" upper="${hip_right_limit}" effort="20" velocity="1.5"/>
-            <dynamics damping="0.5" friction="0.3"/>
+            <limit lower="${hip_left_limit}" upper="${hip_right_limit}" effort="20" velocity="10"/>
         </joint>
         <joint name="${name}_hip_joint2" type="revolute">
@@ -117,22 +123,19 @@
             <origin xyz="0 0 0" rpy="0 0 0"/>
             <axis xyz="0 1 0"/>
-            <limit lower="-1.57" upper="1.57" effort="20" velocity="1.5"/>
-            <dynamics damping="0.5" friction="0.3"/>
+            <limit lower="-1.57" upper="1.57" effort="20" velocity="10"/>
         </joint>
         <joint name="${name}_knee_joint" type="revolute">
             <parent link="${name}_thigh"/>
             <child link="${name}_shin"/>
-            <origin xyz="0 0 -0.1" rpy="0 0 0"/>
+            <origin xyz="0 0 ${-thigh_len}" rpy="0 0 0"/>
             <axis xyz="0 1 0"/>
-            <limit lower="0.0" upper="1.57" effort="20" velocity="1"/>
-            <dynamics damping="0.5" friction="0.3"/>
+            <limit lower="0.0" upper="1.57" effort="20" velocity="10"/>
         </joint>
         <joint name="${name}_ankle_joint1" type="revolute">
             <parent link="${name}_shin"/>
             <child link="${name}_ankle_link"/>
-            <origin xyz="0 0 -0.1" rpy="0 0 0"/>
+            <origin xyz="0 0 ${-shin_len}" rpy="0 0 0"/>
             <axis xyz="0 1 0"/>
-            <limit lower="-1.05" upper="0.52" effort="20" velocity="1"/>
-            <dynamics damping="0.5" friction="0.3"/>
+            <limit lower="-1.05" upper="0.52" effort="20" velocity="10"/>
         </joint>
         <joint name="${name}_ankle_joint2" type="revolute">
@@ -141,9 +144,8 @@
             <origin xyz="0 0 0" rpy="0 0 0"/>
             <axis xyz="1 0 0"/>
-            <limit lower="-0.52" upper="0.52" effort="20" velocity="1"/>
-            <dynamics damping="0.5" friction="0.3"/>
+            <limit lower="-0.52" upper="0.52" effort="20" velocity="10"/>
         </joint>
 	</xacro:macro>
-	<xacro:leg name="left" shift="0.04" hip_left_limit="-0.26" hip_right_limit="0.78"/>
-	<xacro:leg name="right" shift="-0.04" hip_left_limit="-0.78" hip_right_limit="0.26"/>
+	<xacro:leg name="left" shift="${torso_width/2}" hip_left_limit="-0.26" hip_right_limit="0.78"/>
+	<xacro:leg name="right" shift="${-torso_width/2}" hip_left_limit="-0.78" hip_right_limit="0.26"/>
 </robot>

File: urdf/gazebo_bipedal_robot.urdf.xacro (robot description, xacro)
@@ -19,4 +19,11 @@
         </transmission>
 	</xacro:macro>
+	<xacro:macro name="contact" params="link">
+        <gazebo reference="${link}">
+            <mu1>100000.0</mu1>
+            <mu2>100000.0</mu2>
+            <material>Gazebo/White</material>
+        </gazebo>
+	</xacro:macro>
 	<xacro:transmission joint="left_hip_joint1"/>
 	<xacro:transmission joint="left_hip_joint2"/>
@@ -29,4 +36,11 @@
 	<xacro:transmission joint="right_ankle_joint1"/>
 	<xacro:transmission joint="right_ankle_joint2"/>
+	<xacro:contact link="base_link"/>
+	<xacro:contact link="left_thigh"/>
+	<xacro:contact link="left_shin"/>
+	<xacro:contact link="left_foot"/>
+	<xacro:contact link="left_thigh"/>
+	<xacro:contact link="left_shin"/>
+	<xacro:contact link="left_foot"/>
     <gazebo>
         <plugin name="gazebo_ros_control" filename="libgazebo_ros_control.so">
@@ -46,3 +60,15 @@
         </sensor>
     </gazebo>
+    <gazebo reference="right_foot">
+        <sensor name="right_foot_sensor" type="contact">
+            <always_on>true</always_on>
+            <contact>
+                <collision>right_foot_collision_collision</collision>
+            </contact>
+            <plugin name="right_foot_plugin" filename="libgazebo_ros_bumper.so">
+                <bumperTopicName>right_foot_contact</bumperTopicName>
+                <frameName>right_foot</frameName>
+            </plugin>
+        </sensor>
+    </gazebo>
 </robot>

Commit message: Fixed reload bug that makes JointListener return same values

File: urdf/core_bipedal_robot.urdf.xacro (robot description, xacro)
@@ -117,4 +117,5 @@
             <axis xyz="1 0 0"/>
             <limit lower="${hip_left_limit}" upper="${hip_right_limit}" effort="20" velocity="10"/>
+            <dynamics damping="0.02" friction="0.1"/>
         </joint>
         <joint name="${name}_hip_joint2" type="revolute">
@@ -124,4 +125,5 @@
             <axis xyz="0 1 0"/>
             <limit lower="-1.57" upper="1.57" effort="20" velocity="10"/>
+            <dynamics damping="0.02" friction="0.1"/>
         </joint>
         <joint name="${name}_knee_joint" type="revolute">
@@ -131,4 +133,5 @@
             <axis xyz="0 1 0"/>
             <limit lower="0.0" upper="1.57" effort="20" velocity="10"/>
+            <dynamics damping="0.02" friction="0.1"/>
         </joint>
         <joint name="${name}_ankle_joint1" type="revolute">
@@ -138,4 +141,5 @@
             <axis xyz="0 1 0"/>
             <limit lower="-1.05" upper="0.52" effort="20" velocity="10"/>
+            <dynamics damping="0.02" friction="0.1"/>
         </joint>
         <joint name="${name}_ankle_joint2" type="revolute">
@@ -145,4 +149,5 @@
             <axis xyz="1 0 0"/>
             <limit lower="-0.52" upper="0.52" effort="20" velocity="10"/>
+            <dynamics damping="0.02" friction="0.1"/>
         </joint>
 	</xacro:macro>

File: urdf/gazebo_bipedal_robot.urdf.xacro (robot description, xacro)
@@ -21,6 +21,6 @@
 	<xacro:macro name="contact" params="link">
         <gazebo reference="${link}">
-            <mu1>100000.0</mu1>
-            <mu2>100000.0</mu2>
+            <mu1>0.08</mu1>
+            <mu2>0.08</mu2>
             <material>Gazebo/White</material>
         </gazebo>
@@ -54,5 +54,5 @@
                 <collision>left_foot_collision_collision</collision>
             </contact>
-            <plugin name="left_foot_plugin" filename="libgazebo_ros_bumper.so">
+            <plugin name="gazebo_ros_bumper_plugin" filename="libgazebo_ros_bumper.so">
                 <bumperTopicName>left_foot_contact</bumperTopicName>
                 <frameName>left_foot</frameName>
@@ -66,5 +66,5 @@
                 <collision>right_foot_collision_collision</collision>
             </contact>
-            <plugin name="right_foot_plugin" filename="libgazebo_ros_bumper.so">
+            <plugin name="gazebo_ros_bumper_plugin" filename="libgazebo_ros_bumper.so">
                 <bumperTopicName>right_foot_contact</bumperTopicName>
                 <frameName>right_foot</frameName>

Commit message: Minor changes

File: urdf/core_bipedal_robot.urdf.xacro (robot description, xacro)
@@ -1,5 +1,5 @@
 <?xml version="1.0"?>
 <robot name="bipedal_robot" xmlns:xacro="http://www.ros.org/wiki/xacro">
-    <xacro:property name="torso_height" value="0.7"/>
+    <xacro:property name="torso_height" value="0.8"/>
     <xacro:property name="torso_width" value="0.7"/>
     <xacro:property name="thigh_len" value="0.6"/>
@@ -11,5 +11,5 @@
 			<origin xyz="0 0 0" rpy="0 0 0"/>
 			<geometry>
-				<box size="0.3 ${torso_width} ${torso_height}"/>
+				<box size="0.45 ${torso_width} ${torso_height}"/>
 			</geometry>
 			<material name="blue">
@@ -24,5 +24,5 @@
 		</collision>
 		<inertial>
-            <mass value="1.5"/>
+            <mass value="1.1"/>
 		    <origin xyz="0 0 0"/>
 		    <inertia ixx="0.1" ixy="0.0" ixz="0.0" iyy="0.1" iyz="0.0" izz="0.1"/>
@@ -55,5 +55,5 @@
             </collision>
             <inertial>
-                <mass value="2.5"/>
+                <mass value="1.9"/>
                 <origin xyz="0 0 0"/>
                 <inertia ixx="0.1" ixy="0.0" ixz="0.0" iyy="0.1" iyz="0.0" izz="0.1"/>
@@ -77,5 +77,5 @@
             </collision>
             <inertial>
-                <mass value="2"/>
+                <mass value="1.3"/>
                 <origin xyz="0 0 0"/>
                 <inertia ixx="0.1" ixy="0.0" ixz="0.0" iyy="0.1" iyz="0.0" izz="0.1"/>
@@ -93,5 +93,5 @@
                 <origin xyz="0 0 ${-foot_thickness/2}" rpy="0 0 0"/>
                 <geometry>
-                    <box size="0.45 0.3 ${foot_thickness}" />
+                    <box size="0.6 0.5 ${foot_thickness}" />
                 </geometry>
                 <material name="blue">
@@ -102,9 +102,9 @@
                 <origin xyz="0 0 ${-foot_thickness/2}" rpy="0 0 0"/>
                 <geometry>
-                    <box size="0.45 0.3 ${foot_thickness}" />
+                    <box size="0.6 0.5 ${foot_thickness}" />
                 </geometry>
             </collision>
             <inertial>
-                <mass value="1"/>
+                <mass value="1.3"/>
                 <origin xyz="0 0 0"/>
                 <inertia ixx="0.1" ixy="0.0" ixz="0.0" iyy="0.1" iyz="0.0" izz="0.1"/>
@@ -114,8 +114,8 @@
             <parent link="base_link"/>
             <child link="${name}_hip_link"/>
-            <origin xyz="0 ${shift} ${-torso_height/2}" rpy="0 0 0"/>
-            <axis xyz="1 0 0"/>
-            <limit lower="${hip_left_limit}" upper="${hip_right_limit}" effort="20" velocity="10"/>
-            <dynamics damping="0.02" friction="0.1"/>
+            <origin xyz="0 ${shift} ${-torso_height/2+0.2}" rpy="0 0 0"/>
+            <axis xyz="0 1 0"/>
+            <limit lower="-1.57" upper="0.26" effort="20" velocity="10"/>
+            <dynamics damping="0.3" friction="0.07"/>
         </joint>
         <joint name="${name}_hip_joint2" type="revolute">
@@ -123,7 +123,7 @@
             <child link="${name}_thigh"/>
             <origin xyz="0 0 0" rpy="0 0 0"/>
-            <axis xyz="0 1 0"/>
-            <limit lower="-1.57" upper="1.57" effort="20" velocity="10"/>
-            <dynamics damping="0.02" friction="0.1"/>
+            <axis xyz="1 0 0"/>
+            <limit lower="${hip_left_limit}" upper="${hip_right_limit}" effort="20" velocity="10"/>
+            <dynamics damping="0.3" friction="0.07"/>
         </joint>
         <joint name="${name}_knee_joint" type="revolute">
@@ -133,5 +133,5 @@
             <axis xyz="0 1 0"/>
             <limit lower="0.0" upper="1.57" effort="20" velocity="10"/>
-            <dynamics damping="0.02" friction="0.1"/>
+            <dynamics damping="0.2" friction="0"/>
         </joint>
         <joint name="${name}_ankle_joint1" type="revolute">
@@ -140,6 +140,6 @@
             <origin xyz="0 0 ${-shin_len}" rpy="0 0 0"/>
             <axis xyz="0 1 0"/>
-            <limit lower="-1.05" upper="0.52" effort="20" velocity="10"/>
-            <dynamics damping="0.02" friction="0.1"/>
+            <limit lower="-1.05" upper="0.52" effort="10" velocity="10"/>
+            <dynamics damping="0.05" friction="0"/>
         </joint>
         <joint name="${name}_ankle_joint2" type="revolute">
@@ -148,6 +148,6 @@
             <origin xyz="0 0 0" rpy="0 0 0"/>
             <axis xyz="1 0 0"/>
-            <limit lower="-0.52" upper="0.52" effort="20" velocity="10"/>
-            <dynamics damping="0.02" friction="0.1"/>
+            <limit lower="-0.52" upper="0.52" effort="10" velocity="10"/>
+            <dynamics damping="0.05" friction="0"/>
         </joint>
 	</xacro:macro>

File: urdf/full_bipedal_robot.urdf (robot description, URDF)
Before this commit: robot bipedal_robot, 12 links, 11 joints
Links:
- link base_link: mass 0.16 -> 0.9; geometry collision box size=0.3 0.7 0.8; visual box size=0.45 0.7 0.8
- link left_foot: mass 0.02 -> 1.45; geometry collision box size=0.55 0.4 0.08; visual box size=0.55 0.4 0.08
- link left_shin: mass 0.16 -> 1.3; geometry collision cylinder length=0.6 radius=0.07; visual cylinder length=0.6 radius=0.07
- link left_thigh: mass 0.16 -> 1.9; geometry collision cylinder length=0.6 radius=0.07; visual cylinder length=0.6 radius=0.07
- link right_foot: mass 0.02 -> 1.45; geometry collision box size=0.55 0.4 0.08; visual box size=0.55 0.4 0.08
- link right_shin: mass 0.16 -> 1.3; geometry collision cylinder length=0.6 radius=0.07; visual cylinder length=0.6 radius=0.07
- link right_thigh: mass 0.16 -> 1.9; geometry collision cylinder length=0.6 radius=0.07; visual cylinder length=0.6 radius=0.07
Joints:
- joint left_ankle_joint1: limit lower=-1.57 upper=1.57 effort=20 velocity=1 -> lower=-1.05 upper=0.52 effort=20 velocity=10; origin xyz=0 0 -0.1 rpy=0 0 0 -> xyz=0 0 -0.6 rpy=0 0 0
- joint left_ankle_joint2: limit lower=-1.57 upper=1.57 effort=20 velocity=1 -> lower=-0.52 upper=0.52 effort=20 velocity=10; origin xyz=0 0 -0.1 rpy=0 0 0 -> xyz=0 0 0 rpy=0 0 0
- joint left_hip_joint1: axis 1 0 0 -> 0 1 0; limit lower=-1.57 upper=1.57 effort=20 velocity=1.5 -> lower=-1.57 upper=0.26 effort=20 velocity=10; origin xyz=0 0.04 -0.03 rpy=0 0 0 -> xyz=0 0.35 -0.2 rpy=0 0 0
- joint left_hip_joint2: axis 0 1 0 -> 1 0 0; limit lower=-1.57 upper=1.57 effort=20 velocity=1.5 -> lower=-0.26 upper=0.78 effort=20 velocity=10; origin xyz=0 0 -0.03 rpy=0 0 0 -> xyz=0 0 0 rpy=0 0 0
- joint left_knee_joint: limit lower=0.0 upper=1.57 effort=20 velocity=1 -> lower=0.0 upper=1.57 effort=20 velocity=10; origin xyz=0 0 -0.1 rpy=0 0 0 -> xyz=0 0 -0.6 rpy=0 0 0
- joint right_ankle_joint1: limit lower=-1.57 upper=1.57 effort=20 velocity=1 -> lower=-1.05 upper=0.52 effort=20 velocity=10; origin xyz=0 0 -0.1 rpy=0 0 0 -> xyz=0 0 -0.6 rpy=0 0 0
- joint right_ankle_joint2: limit lower=-1.57 upper=1.57 effort=20 velocity=1 -> lower=-0.52 upper=0.52 effort=20 velocity=10; origin xyz=0 0 -0.1 rpy=0 0 0 -> xyz=0 0 0 rpy=0 0 0
- joint right_hip_joint1: axis 1 0 0 -> 0 1 0; limit lower=-1.57 upper=1.57 effort=20 velocity=1.5 -> lower=-1.57 upper=0.26 effort=20 velocity=10; origin xyz=0 -0.04 -0.03 rpy=0 0 0 -> xyz=0 -0.35 -0.2 rpy=0 0 0
- joint right_hip_joint2: axis 0 1 0 -> 1 0 0; limit lower=-1.57 upper=1.57 effort=20 velocity=1.5 -> lower=-0.78 upper=0.26 effort=20 velocity=10; origin xyz=0 0 -0.03 rpy=0 0 0 -> xyz=0 0 0 rpy=0 0 0
- joint right_knee_joint: limit lower=0.0 upper=1.57 effort=20 velocity=1 -> lower=0.0 upper=1.57 effort=20 velocity=10; origin xyz=0 0 -0.1 rpy=0 0 0 -> xyz=0 0 -0.6 rpy=0 0 0

File: urdf/gazebo_bipedal_robot.urdf.xacro (robot description, xacro)
@@ -21,7 +21,8 @@
 	<xacro:macro name="contact" params="link">
         <gazebo reference="${link}">
-            <mu1>0.08</mu1>
-            <mu2>0.08</mu2>
-            <material>Gazebo/White</material>
+            <mu1>1.0</mu1>
+            <mu2>1.0</mu2>
+            <minDepth>0.01</minDepth>
+            <maxVel value="20.0"/>
         </gazebo>
 	</xacro:macro>
@@ -40,7 +41,7 @@
 	<xacro:contact link="left_shin"/>
 	<xacro:contact link="left_foot"/>
-	<xacro:contact link="left_thigh"/>
-	<xacro:contact link="left_shin"/>
-	<xacro:contact link="left_foot"/>
+	<xacro:contact link="right_thigh"/>
+	<xacro:contact link="right_shin"/>
+	<xacro:contact link="right_foot"/>
     <gazebo>
         <plugin name="gazebo_ros_control" filename="libgazebo_ros_control.so">
