Commit message: Minor changes

File: urdf/core_bipedal_robot.urdf.xacro (robot description, xacro)
@@ -116,5 +116,5 @@
             <origin xyz="0 ${shift} ${-torso_height/2+0.2}" rpy="0 0 0"/>
             <axis xyz="0 1 0"/>
-            <limit lower="-1.57" upper="0.26" effort="20" velocity="10"/>
+            <limit lower="-1.57" upper="0.52" effort="50" velocity="10"/>
             <dynamics damping="0.3" friction="0.07"/>
         </joint>
@@ -124,5 +124,5 @@
             <origin xyz="0 0 0" rpy="0 0 0"/>
             <axis xyz="1 0 0"/>
-            <limit lower="${hip_left_limit}" upper="${hip_right_limit}" effort="20" velocity="10"/>
+            <limit lower="${hip_left_limit}" upper="${hip_right_limit}" effort="50" velocity="10"/>
             <dynamics damping="0.3" friction="0.07"/>
         </joint>
@@ -132,5 +132,5 @@
             <origin xyz="0 0 ${-thigh_len}" rpy="0 0 0"/>
             <axis xyz="0 1 0"/>
-            <limit lower="0.0" upper="1.57" effort="20" velocity="10"/>
+            <limit lower="-0.17" upper="1.57" effort="50" velocity="10"/>
             <dynamics damping="0.2" friction="0"/>
         </joint>
@@ -140,6 +140,6 @@
             <origin xyz="0 0 ${-shin_len}" rpy="0 0 0"/>
             <axis xyz="0 1 0"/>
-            <limit lower="-1.05" upper="0.52" effort="10" velocity="10"/>
-            <dynamics damping="0.05" friction="0"/>
+            <limit lower="-1.05" upper="0.52" effort="30" velocity="10"/>
+            <dynamics friction="0"/>
         </joint>
         <joint name="${name}_ankle_joint2" type="revolute">
@@ -148,6 +148,6 @@
             <origin xyz="0 0 0" rpy="0 0 0"/>
             <axis xyz="1 0 0"/>
-            <limit lower="-0.52" upper="0.52" effort="10" velocity="10"/>
-            <dynamics damping="0.05" friction="0"/>
+            <limit lower="-0.52" upper="0.52" effort="30" velocity="10"/>
+            <dynamics friction="0"/>
         </joint>
 	</xacro:macro>

File: urdf/full_bipedal_robot.urdf (robot description, URDF)
Before this commit: robot bipedal_robot, 12 links, 11 joints
Links:
- link base_link: mass 0.9 -> 1.1
- link left_foot: mass 1.45 -> 1.3; geometry collision box size=0.6 0.5 0.08; visual box size=0.6 0.5 0.08
- link right_foot: mass 1.45 -> 1.3; geometry collision box size=0.6 0.5 0.08; visual box size=0.6 0.5 0.08
Joints:
- joint left_ankle_joint1: limit lower=-1.05 upper=0.52 effort=20 velocity=10 -> lower=-1.05 upper=0.52 effort=30 velocity=10
- joint left_ankle_joint2: limit lower=-0.52 upper=0.52 effort=20 velocity=10 -> lower=-0.52 upper=0.52 effort=30 velocity=10
- joint left_hip_joint1: limit lower=-1.57 upper=0.26 effort=20 velocity=10 -> lower=-1.57 upper=0.52 effort=50 velocity=10
- joint left_hip_joint2: limit lower=-0.26 upper=0.78 effort=20 velocity=10 -> lower=-0.26 upper=0.78 effort=50 velocity=10
- joint left_knee_joint: limit lower=0.0 upper=1.57 effort=20 velocity=10 -> lower=-0.17 upper=1.57 effort=50 velocity=10
- joint right_ankle_joint1: limit lower=-1.05 upper=0.52 effort=20 velocity=10 -> lower=-1.05 upper=0.52 effort=30 velocity=10
- joint right_ankle_joint2: limit lower=-0.52 upper=0.52 effort=20 velocity=10 -> lower=-0.52 upper=0.52 effort=30 velocity=10
- joint right_hip_joint1: limit lower=-1.57 upper=0.26 effort=20 velocity=10 -> lower=-1.57 upper=0.52 effort=50 velocity=10
- joint right_hip_joint2: limit lower=-0.78 upper=0.26 effort=20 velocity=10 -> lower=-0.78 upper=0.26 effort=50 velocity=10
- joint right_knee_joint: limit lower=0.0 upper=1.57 effort=20 velocity=10 -> lower=-0.17 upper=1.57 effort=50 velocity=10

File: urdf/gazebo_bipedal_robot.urdf.xacro (robot description, xacro)
@@ -21,10 +21,30 @@
 	<xacro:macro name="contact" params="link">
         <gazebo reference="${link}">
-            <mu1>1.0</mu1>
-            <mu2>1.0</mu2>
-            <minDepth>0.01</minDepth>
-            <maxVel value="20.0"/>
+            <mu1>10000.0</mu1>
+            <mu2>10000.0</mu2>
+            <minDepth>0.001</minDepth>
+            <maxVel value="0.0"/>
         </gazebo>
 	</xacro:macro>
+	<gazebo reference="right_foot">
+	    <collision name='right_foot_collision_collision'>
+	        <surface>
+                <bounce>
+                    <restitution_coefficient>0.9</restitution_coefficient>
+                    <threshold>0.0</threshold>
+                </bounce>
+            </surface>
+	    </collision>
+	</gazebo>
+	<gazebo reference="left_foot">
+	    <collision name='left_foot_collision_collision'>
+	        <surface>
+                <bounce>
+                    <restitution_coefficient>0.9</restitution_coefficient>
+                    <threshold>0.0</threshold>
+                </bounce>
+            </surface>
+	    </collision>
+	</gazebo>
 	<xacro:transmission joint="left_hip_joint1"/>
 	<xacro:transmission joint="left_hip_joint2"/>
